Commit message: robot hardware (wip)

File: mecanumbot_description/urdf/mecanumbot.urdf (robot description, URDF)
Before this commit: robot mecanumbot, 6 links, 5 joints
Joints:
- joint rl_wheel_joint: type fixed -> continuous
- joint rr_wheel_joint: type fixed -> continuous

Commit message: Update robot description to position wheels
Signed-off-by: Randy Deborggraeve <randy@deb-ict.com>

File: mecanumbot_description/urdf/mecanumbot.urdf (robot description, URDF)
Before this commit: robot mecanumbot, 6 links, 5 joints
Links:
- link fr_wheel_link: geometry collision box size=${wheel_width} ${wheel_radius*2} ${wheel_radius*2}; visual mesh filename=package://mecanumbot_description/meshes/fr_wheel_link.STL scale=0.6 0.6 0.6
- link rl_wheel_link: geometry collision box size=${wheel_width} ${wheel_radius*2} ${wheel_radius*2}; visual mesh filename=package://mecanumbot_description/meshes/rl_wheel_link.STL scale=0.6 0.6 0.6
- link rr_wheel_link: geometry collision box size=${wheel_width} ${wheel_radius*2} ${wheel_radius*2}; visual mesh filename=package://mecanumbot_description/meshes/rr_wheel_link.STL scale=0.6 0.6 0.6
Joints:
- joint fr_wheel_joint: axis (none) -> -1 0 0; origin xyz=-0.19 0.23 ${wheel_offset_z} rpy=0 0 0 -> xyz=${-wheel_offset_x} ${wheel_offset_y} ${wheel_offset_z} rpy=0 0 ${-M_PI/2}
- joint rl_wheel_joint: axis (none) -> -1 0 0; origin xyz=0.19 -0.23 ${wheel_offset_z} rpy=0 0 0 -> xyz=${wheel_offset_x} ${-wheel_offset_y} ${wheel_offset_z} rpy=0 0 ${-M_PI/2}
- joint rr_wheel_joint: axis (none) -> -1 0 0; origin xyz=0.19 0.23 ${wheel_offset_z} rpy=0 0 0 -> xyz=${wheel_offset_x} ${wheel_offset_y} ${wheel_offset_z} rpy=0 0 ${-M_PI/2}

Commit message: Make all wheels visible
Signed-off-by: Randy Deborggraeve <randy@deb-ict.com>

File: mecanumbot_description/urdf/mecanumbot.urdf (robot description, URDF)
Before this commit: robot mecanumbot, 6 links, 5 joints
Joints:
- joint fl_wheel_joint: axis -1 0 0 -> 1 0 0
- joint fr_wheel_joint: origin xyz=${-wheel_offset_x} ${wheel_offset_y} ${wheel_offset_z} rpy=0 0 ${-M_PI/2} -> xyz=${-wheel_offset_x} ${wheel_offset_y} ${wheel_offset_z} rpy=0 0 ${M_PI/2}
- joint rr_wheel_joint: origin xyz=${wheel_offset_x} ${wheel_offset_y} ${wheel_offset_z} rpy=0 0 ${-M_PI/2} -> xyz=${wheel_offset_x} ${wheel_offset_y} ${wheel_offset_z} rpy=0 0 ${M_PI/2}

Commit message: Fix rl wheel direction
Signed-off-by: Randy Deborggraeve <randy@deb-ict.com>

File: mecanumbot_description/urdf/mecanumbot.urdf (robot description, URDF)
Before this commit: robot mecanumbot, 6 links, 5 joints
Joints:
- joint rl_wheel_joint: axis -1 0 0 -> 1 0 0
